File: Optical Interrupter/optical interrupter V1.brd (EAGLE design)
At the start: 160 x 100 mm, 27 parts, among them IC1 NE555, Q1 2n2222a, Q2 2n2222a, Q3 2n2222a, SW1 EC12E_SW, U1 MIC4426YN

Commit message: updated file structure
Parts:
- removed Q1, Q2, Q3: 2n2222a, transistor-npn:TO92-EBC
- added JP1, JP2: (no value), pinhead:1X02
- added JP3, JP4: (no value), pinhead:1X04
- added T1, T2, T3: 2N2222, adafruit:TO92-EBC-OVAL
- moved S1 48.1 mm to (-15.7, 32.8)
- moved S2 48.1 mm to (-16.5, 24.4)
- moved SW1 48.1 mm to (-29.5, 28.7)
- moved R10 2.54 mm to (63.5, 34.3)
Connections:
- new net N$30: JP4.1, SW1.A
- new net N$31: JP4.3, SW1.D
- new net N$32: JP1.1, S1.2
- new net N$33: JP1.2, S2.4
- new net SW1: JP2.2, U$1.11
- new net SW2: JP2.1, U$1.12
- net 5V: now also T1.E, T2.E, T3.E
- net GND: now also JP3.1; no longer Q1.E, Q2.E, Q3.E, SW1.A
- net N$14: now also JP4.2, SW1.E; no longer S1.2, U$1.11
- net N$15: now also JP4.4, SW1.B; no longer S2.4, U$1.12
- net N$16: now also JP3.4; no longer SW1.B
- net N$19: now also JP3.3; no longer SW1.D
- net N$20: now also JP3.2; no longer SW1.E
- net N$4: now also T2.B; no longer Q1.B
- net N$5: now also T3.B; no longer Q3.B
- net N$6: now also T1.B; no longer Q2.B
- net N$7: now also T1.C, T2.C, T3.C; no longer Q1.C, Q2.C, Q3.C
Routing:
- net GND: track 104.5 -> 187.5 mm
- net N$16: track 0.00 -> 40.6 mm
- net N$19: track 2.54 -> 25.4 mm
- net N$20: track 2.54 -> 20.8 mm
- net SW1: track 0.00 -> 17.8 mm
- net N$7: track 50.8 -> 33.0 mm
- net SW2: track 0.00 -> 12.7 mm
- net 5V: track 12.7 -> 10.2 mm
- net N$6: track 2.54 -> 0.00 mm
- net N$5: track 2.54 -> 0.00 mm
- net N$4: track 2.54 -> 0.00 mm
- net N$12: track 13.6 -> 12.6 mm
